Commit message: Update URDF: Refactor standoff macro and update LiDAR mount (Issue #2)
- Made standoff.xacro macro reusable with length and z parameters
- Replaced manual standoff placements with the new macro
- Updated LiDAR Z offset to 0.194 to account for 80mm M2.5 spacer and 40mm sensor offset
- Added 4 x 80mm standoffs for the LiDAR mount
- Updated chassis mass and inertia tensors to reflect 1.976kg total vehicle weight

File: src/vehicle_description/urdf/standoff.xacro (robot description, xacro)
@@ -1,10 +1,10 @@
 <?xml version="1.0"?>
 <robot xmlns:xacro="http://www.ros.org/wiki/xacro">
-  <!-- 황동 지지대 하나: 지름 5 mm, 길이 50 mm -->
-  <xacro:macro name="standoff" params="x y">
+  <!-- 원통형 지지대 매크로 -->
+  <xacro:macro name="standoff" params="x y z length">
     <visual>
-      <origin xyz="${x} ${y} 0.047" rpy="0 0 0"/>
+      <origin xyz="${x} ${y} ${z}" rpy="0 0 0"/>
       <geometry>
-        <cylinder radius="0.0025" length="0.050"/>
+        <cylinder radius="0.0025" length="${length}"/>
       </geometry>
       <material name="brass">
@@ -13,7 +13,7 @@
     </visual>
     <collision>
-      <origin xyz="${x} ${y} 0.047" rpy="0 0 0"/>
+      <origin xyz="${x} ${y} ${z}" rpy="0 0 0"/>
       <geometry>
-        <cylinder radius="0.0025" length="0.050"/>
+        <cylinder radius="0.0025" length="${length}"/>
       </geometry>
     </collision>

File: src/vehicle_description/urdf/vehicle.urdf.xacro (robot description, xacro)
@@ -43,11 +43,17 @@
       </geometry>
     </collision>
-    <!-- 황동 지지대 6개: X·Y는 실제 체결 구멍 확인 전 임시 좌표 -->
-    <xacro:standoff x="0.100"  y="0.045"/>
-    <xacro:standoff x="0.100"  y="-0.045"/>
-    <xacro:standoff x="0.000"  y="0.045"/>
-    <xacro:standoff x="0.000"  y="-0.045"/>
-    <xacro:standoff x="-0.100" y="0.045"/>
-    <xacro:standoff x="-0.100" y="-0.045"/>
+    <!-- 황동 지지대 6개 (섀시 상/하판 고정용, 길이 50mm) -->
+    <xacro:standoff x="0.100"  y="0.045"  z="0.047" length="0.050"/>
+    <xacro:standoff x="0.100"  y="-0.045" z="0.047" length="0.050"/>
+    <xacro:standoff x="0.000"  y="0.045"  z="0.047" length="0.050"/>
+    <xacro:standoff x="0.000"  y="-0.045" z="0.047" length="0.050"/>
+    <xacro:standoff x="-0.100" y="0.045"  z="0.047" length="0.050"/>
+    <xacro:standoff x="-0.100" y="-0.045" z="0.047" length="0.050"/>
+    <!-- 라이다용 80mm M2.5 스페이서 4개 (상판 Z=0.074 부터 Z=0.154 까지, 중심 0.114) -->
+    <!-- 라이다 중심(x=0.030, y=0.000) 기준으로 가로세로 약 30mm 간격(±0.015)으로 배치 -->
+    <xacro:standoff x="0.045"  y="0.015"  z="0.114" length="0.080"/>
+    <xacro:standoff x="0.045"  y="-0.015" z="0.114" length="0.080"/>
+    <xacro:standoff x="0.015"  y="0.015"  z="0.114" length="0.080"/>
+    <xacro:standoff x="0.015"  y="-0.015" z="0.114" length="0.080"/>
     <inertial>
       <origin xyz="0 0 0.047" rpy="0 0 0"/>
@@ -104,5 +110,5 @@
   <xacro:imu parent="base_link" x="-0.050" y="0" z="0.074"/>
   <!-- 라이다 스캔 평면: 차체 중심보다 앞쪽 30 mm -->
-  <xacro:lidar parent="base_link" x="0.030" y="0" z="0.174"/>
+  <xacro:lidar parent="base_link" x="0.030" y="0" z="0.194"/>
   <!-- 상판 전방 95 mm에 팬·틸트 카메라 조립 -->
   <xacro:camera parent="base_link" x="0.095" y="0" z="0.074"/>
