Commit message: feat(description): align vehicle URDF with chassis meshes

File: src/vehicle_description/urdf/gazebo.xacro (robot description, xacro)
@@ -11,5 +11,5 @@
       <right_joint>front_right_wheel_joint</right_joint>
       <right_joint>rear_right_wheel_joint</right_joint>
-      <wheel_separation>0.150</wheel_separation>
+      <wheel_separation>${wheel_separation}</wheel_separation>
       <wheel_radius>${wheel_radius}</wheel_radius>
       <topic>/cmd_vel</topic>

File: src/vehicle_description/urdf/standoff.xacro (robot description, xacro)
@@ -2,14 +2,16 @@
 <robot xmlns:xacro="http://www.ros.org/wiki/xacro">
   <!-- 원통형 지지대 매크로 -->
-  <xacro:macro name="standoff" params="x y z length">
-    <visual>
-      <origin xyz="${x} ${y} ${z}" rpy="0 0 0"/>
-      <geometry>
-        <cylinder radius="0.0025" length="${length}"/>
-      </geometry>
-      <material name="brass">
-        <color rgba="0.75 0.55 0.20 1.0"/>
-      </material>
-    </visual>
+  <xacro:macro name="standoff" params="x y z length show_visual:=true">
+    <xacro:if value="${show_visual}">
+      <visual>
+        <origin xyz="${x} ${y} ${z}" rpy="0 0 0"/>
+        <geometry>
+          <cylinder radius="0.0025" length="${length}"/>
+        </geometry>
+        <material name="brass">
+          <color rgba="0.75 0.55 0.20 1.0"/>
+        </material>
+      </visual>
+    </xacro:if>
     <collision>
       <origin xyz="${x} ${y} ${z}" rpy="0 0 0"/>

File: src/vehicle_description/urdf/vehicle.urdf.xacro (robot description, xacro)
@@ -1,5 +1,15 @@
 <?xml version="1.0"?>
 <robot xmlns:xacro="http://www.ros.org/wiki/xacro" name="vehicle">
-  <xacro:property name="wheel_radius" value="0.0325"/>
+  <!-- four-wheel-drvie-main-body.stl 기준, 단위 m. 원본 -Z가 전방, 네 바퀴 축의 중심이 원점. -->
+  <xacro:property name="wheel_radius" value="0.0335"/>
+  <xacro:property name="wheel_width" value="0.027"/>
+  <xacro:property name="wheel_separation" value="0.1203"/>
+  <xacro:property name="wheelbase" value="0.0994"/>
+  <xacro:property name="chassis_center_x" value="-0.006"/>
+  <xacro:property name="lower_plate_z" value="0.02565"/>
+  <xacro:property name="upper_plate_z" value="0.06765"/>
+  <xacro:property name="plate_thickness" value="0.002"/>
+  <xacro:property name="lower_plate_top" value="${lower_plate_z + plate_thickness / 2}"/>
+  <xacro:property name="upper_plate_top" value="${upper_plate_z + plate_thickness / 2}"/>
   <xacro:include filename="wheel.xacro"/>
   <xacro:include filename="standoff.xacro"/>
@@ -19,57 +29,73 @@
   <!-- 섀시 -->
   <link name="chassis_link">
-    <!-- 섀시 하판 (Lower Plate): 228 × 110 × 2 mm -->
+    <!-- 상·하판, 지지대, 모터와 체결 부품. 바퀴/허브는 회전 링크에 분리. -->
     <visual>
-      <origin xyz="0 0 0.021" rpy="0 0 0"/>
       <geometry>
-        <box size="0.228 0.110 0.002"/>
+        <mesh filename="package://vehicle_description/meshes/chassis_body.stl"/>
       </geometry>
+      <material name="chassis_gray">
+        <color rgba="0.55 0.55 0.55 1"/>
+      </material>
     </visual>
+    <!-- 충돌 계산은 상·하판과 모터의 단순 형상으로 근사. -->
     <collision>
-      <origin xyz="0 0 0.021" rpy="0 0 0"/>
+      <origin xyz="${chassis_center_x} 0 ${lower_plate_z}" rpy="0 0 0"/>
       <geometry>
-        <box size="0.228 0.110 0.002"/>
+        <box size="0.228 0.110 ${plate_thickness}"/>
       </geometry>
     </collision>
     <!-- 섀시 상판 (Upper Plate): 228 × 148 × 2 mm -->
-    <visual>
-      <origin xyz="0 0 0.073" rpy="0 0 0"/>
+    <collision>
+      <origin xyz="${chassis_center_x} 0 ${upper_plate_z}" rpy="0 0 0"/>
       <geometry>
-        <box size="0.228 0.148 0.002"/>
-      </geometry>
-    </visual>
-    <collision>
-      <origin xyz="0 0 0.073" rpy="0 0 0"/>
-      <geometry>
-        <box size="0.228 0.148 0.002"/>
+        <box size="0.228 0.148 ${plate_thickness}"/>
       </geometry>
     </collision>
-    <!-- 황동 지지대 6개 (섀시 상/하판 고정용, 길이 50mm) -->
-    <xacro:standoff x="0.100"  y="0.045"  z="0.047" length="0.050"/>
-    <xacro:standoff x="0.100"  y="-0.045" z="0.047" length="0.050"/>
-    <xacro:standoff x="0.000"  y="0.045"  z="0.047" length="0.050"/>
-    <xacro:standoff x="0.000"  y="-0.045" z="0.047" length="0.050"/>
-    <xacro:standoff x="-0.100" y="0.045"  z="0.047" length="0.050"/>
-    <xacro:standoff x="-0.100" y="-0.045" z="0.047" length="0.050"/>
-    <!-- 라이다용 50mm M2.5 스페이서 4개 (상판 Z=0.074 부터 Z=0.124 까지, 중심 0.099) -->
+    <!-- 모터/기어박스 외접 박스. 축과 작은 체결 부품의 충돌 형상은 생략. -->
+    <collision name="front_left_motor">
+      <origin xyz="0.069 0.02035 0"/>
+      <geometry><box size="0.0644 0.0671 0.038"/></geometry>
+    </collision>
+    <collision name="front_right_motor">
+      <origin xyz="0.0304 -0.02035 0"/>
+      <geometry><box size="0.0644 0.0671 0.038"/></geometry>
+    </collision>
+    <collision name="rear_left_motor">
+      <origin xyz="-0.0304 0.02035 0"/>
+      <geometry><box size="0.0644 0.0671 0.038"/></geometry>
+    </collision>
+    <collision name="rear_right_motor">
+      <origin xyz="-0.069 -0.02035 0"/>
+      <geometry><box size="0.06443 0.0671 0.03808"/></geometry>
+    </collision>
+    <!-- STL 지지대 위치. 판 사이 40 mm 구간의 충돌만 추가하며 외형은 메시 사용. -->
+    <xacro:standoff x="0.096"  y="0.036"  z="${(lower_plate_z + upper_plate_z) / 2}" length="0.040" show_visual="false"/>
+    <xacro:standoff x="0.096"  y="-0.036" z="${(lower_plate_z + upper_plate_z) / 2}" length="0.040" show_visual="false"/>
+    <xacro:standoff x="0.000"  y="0.050"  z="${(lower_plate_z + upper_plate_z) / 2}" length="0.040" show_visual="false"/>
+    <xacro:standoff x="0.000"  y="-0.050" z="${(lower_plate_z + upper_plate_z) / 2}" length="0.040" show_visual="false"/>
+    <xacro:standoff x="-0.100" y="0.036"  z="${(lower_plate_z + upper_plate_z) / 2}" length="0.040" show_visual="false"/>
+    <xacro:standoff x="-0.100" y="-0.036" z="${(lower_plate_z + upper_plate_z) / 2}" length="0.040" show_visual="false"/>
+    <!-- 추가 장착물의 XY 배치는 기존 추정값. 높이는 STL 상판 윗면에 연동. -->
+    <!-- 라이다용 50mm M2.5 스페이서 4개 -->
     <!-- 라이다 중심(x=0.030, y=0.000) 기준으로 가로세로 약 30mm 간격(±0.015)으로 배치 -->
-    <xacro:standoff x="0.045"  y="0.015"  z="0.099" length="0.050"/>
-    <xacro:standoff x="0.045"  y="-0.015" z="0.099" length="0.050"/>
-    <xacro:standoff x="0.015"  y="0.015"  z="0.099" length="0.050"/>
-    <xacro:standoff x="0.015"  y="-0.015" z="0.099" length="0.050"/>
-    <!-- 라즈베리파이5용 20mm M2.5 스페이서 4개 (상판 Z=0.074 부터 Z=0.094 까지, 중심 0.084) -->
+    <xacro:standoff x="0.045"  y="0.015"  z="${upper_plate_top + 0.025}" length="0.050"/>
+    <xacro:standoff x="0.045"  y="-0.015" z="${upper_plate_top + 0.025}" length="0.050"/>
+    <xacro:standoff x="0.015"  y="0.015"  z="${upper_plate_top + 0.025}" length="0.050"/>
+    <xacro:standoff x="0.015"  y="-0.015" z="${upper_plate_top + 0.025}" length="0.050"/>
+    <!-- 라즈베리파이5용 20mm M2.5 스페이서 4개 -->
     <!-- 라즈베리파이 중심(x=-0.060, y=0.040) 기준으로 가로 58mm(±0.029), 세로 49mm(±0.0245) 간격 -->
-    <xacro:standoff x="-0.031" y="0.0645" z="0.084" length="0.020"/>
-    <xacro:standoff x="-0.031" y="0.0155" z="0.084" length="0.020"/>
-    <xacro:standoff x="-0.089" y="0.0645" z="0.084" length="0.020"/>
-    <xacro:standoff x="-0.089" y="0.0155" z="0.084" length="0.020"/>
-    <!-- ESP32 확장보드용 20mm 스페이서 4개 (상판 Z=0.074 부터 Z=0.094 까지, 중심 0.084) -->
+    <xacro:standoff x="-0.031" y="0.0645" z="${upper_plate_top + 0.010}" length="0.020"/>
+    <xacro:standoff x="-0.031" y="0.0155" z="${upper_plate_top + 0.010}" length="0.020"/>
+    <xacro:standoff x="-0.089" y="0.0645" z="${upper_plate_top + 0.010}" length="0.020"/>
+    <xacro:standoff x="-0.089" y="0.0155" z="${upper_plate_top + 0.010}" length="0.020"/>
+    <!-- ESP32 확장보드용 20mm 스페이서 4개 -->
     <!-- 보드 중심(x=-0.060, y=-0.040) 기준으로 대략적인 4모서리(±0.035, ±0.023)에 배치 -->
-    <xacro:standoff x="-0.025" y="-0.017" z="0.084" length="0.020"/>
-    <xacro:standoff x="-0.025" y="-0.063" z="0.084" length="0.020"/>
-    <xacro:standoff x="-0.095" y="-0.017" z="0.084" length="0.020"/>
-    <xacro:standoff x="-0.095" y="-0.063" z="0.084" length="0.020"/>
+    <xacro:standoff x="-0.025" y="-0.017" z="${upper_plate_top + 0.010}" length="0.020"/>
+    <xacro:standoff x="-0.025" y="-0.063" z="${upper_plate_top + 0.010}" length="0.020"/>
+    <xacro:standoff x="-0.095" y="-0.017" z="${upper_plate_top + 0.010}" length="0.020"/>
+    <xacro:standoff x="-0.095" y="-0.063" z="${upper_plate_top + 0.010}" length="0.020"/>
+    <!-- 질량/관성은 기존 추정값 유지. 무게중심은 판 사이 중심으로 근사. -->
     <inertial>
-      <origin xyz="0 0 0.047" rpy="0 0 0"/>
+      <origin xyz="${chassis_center_x} 0 ${(lower_plate_z + upper_plate_z) / 2}" rpy="0 0 0"/>
       <mass value="1.296"/>
       <inertia
@@ -114,20 +140,20 @@
     <parent link="chassis_link" />
     <child link="battery_link" />
-    <origin xyz="0 0 0.041" rpy="0 0 0" />
+    <origin xyz="0 0 ${lower_plate_top + 0.019}" rpy="0 0 0" />
   </joint>
   <!-- 바퀴 4개 -->
-  <xacro:wheel name="front_left"  x="0.065"  y="0.075"/>
-  <xacro:wheel name="front_right" x="0.065"  y="-0.075"/>
-  <xacro:wheel name="rear_left"   x="-0.065" y="0.075"/>
-  <xacro:wheel name="rear_right"  x="-0.065" y="-0.075"/>
+  <xacro:wheel name="front_left"  x="${wheelbase / 2}"  y="${wheel_separation / 2}"/>
+  <xacro:wheel name="front_right" x="${wheelbase / 2}"  y="${-wheel_separation / 2}"/>
+  <xacro:wheel name="rear_left"   x="${-wheelbase / 2}" y="${wheel_separation / 2}"/>
+  <xacro:wheel name="rear_right"  x="${-wheelbase / 2}" y="${-wheel_separation / 2}"/>
   <!-- IMU: 상판 좌측 전방 (10-axis IMU module 홀 위치)에 IMU 장착 -->
-  <xacro:imu parent="base_link" x="0.060" y="0.060" z="0.074"/>
+  <xacro:imu parent="base_link" x="0.060" y="0.060" z="${upper_plate_top}"/>
   <!-- 라이다 스캔 평면: 차체 중심보다 앞쪽 30 mm -->
-  <xacro:lidar parent="base_link" x="0.030" y="0" z="0.164"/>
+  <xacro:lidar parent="base_link" x="0.030" y="0" z="${upper_plate_top + 0.090}"/>
   <!-- 상판 전방 95 mm에 Figure-2 방식으로 카메라 매립: z는 상판 윗면, 위 62 / 아래 16 mm -->
-  <xacro:camera parent="base_link" x="0.095" y="0" z="0.074"/>
+  <xacro:camera parent="base_link" x="0.095" y="0" z="${upper_plate_top}"/>
   <!-- 상판 후방 좌측에 라즈베리파이 5 배치 (20mm 지지대 사용) -->
-  <xacro:raspberry_pi parent="base_link" x="-0.060" y="0.040" z="0.104"/>
+  <xacro:raspberry_pi parent="base_link" x="-0.060" y="0.040" z="${upper_plate_top + 0.030}"/>
   <!-- 상판 후방 우측에 ESP32 + 확장보드 배치 (20mm 지지대 사용) -->
-  <xacro:esp32_board parent="base_link" x="-0.060" y="-0.040" z="0.1015"/>
+  <xacro:esp32_board parent="base_link" x="-0.060" y="-0.040" z="${upper_plate_top + 0.0275}"/>
 </robot>

File: src/vehicle_description/urdf/wheel.xacro (robot description, xacro)
@@ -3,24 +3,28 @@
   <!-- 바퀴 하나의 링크와 조인트를 만드는 매크로 -->
   <xacro:macro name="wheel" params="name x y">
+    <!-- 기존 추정 질량 유지, 관성은 수정된 치수의 균일 원통으로 근사. -->
+    <xacro:property name="wheel_mass" value="0.040"/>
     <link name="${name}_wheel_link">
       <visual>
-        <origin xyz="0 0 0" rpy="1.5708 0 0"/>
         <geometry>
-          <cylinder radius="${wheel_radius}" length="0.026"/>
+          <mesh filename="package://vehicle_description/meshes/${name}_wheel.stl"/>
         </geometry>
+        <material name="wheel_dark_gray">
+          <color rgba="0.12 0.12 0.12 1"/>
+        </material>
       </visual>
       <collision>
-        <origin xyz="0 0 0" rpy="1.5708 0 0"/>
+        <origin xyz="0 0 0" rpy="${pi / 2} 0 0"/>
         <geometry>
-          <cylinder radius="${wheel_radius}" length="0.026"/>
+          <cylinder radius="${wheel_radius}" length="${wheel_width}"/>
         </geometry>
       </collision>
       <inertial>
         <origin xyz="0 0 0" rpy="0 0 0"/>
-        <mass value="0.040"/>
+        <mass value="${wheel_mass}"/>
         <inertia
-          ixx="0.0000128" ixy="0" ixz="0"
-          iyy="0.0000211" iyz="0"
-          izz="0.0000128"/>
+          ixx="${wheel_mass * (3 * wheel_radius**2 + wheel_width**2) / 12}" ixy="0" ixz="0"
+          iyy="${wheel_mass * wheel_radius**2 / 2}" iyz="0"
+          izz="${wheel_mass * (3 * wheel_radius**2 + wheel_width**2) / 12}"/>
       </inertial>
     </link>

Commit message: feat: add simulation lidar with shared YAML configuration

File: src/vehicle_description/urdf/gazebo.xacro (robot description, xacro)
@@ -20,3 +20,42 @@
     </plugin>
   </gazebo>
+  <!-- 시뮬레이션 라이다의 초기 측정 설정 -->
+  <xacro:arg
+    name="lidar_config_file"
+    default="${xacro.abs_filename('../config/lidar.yaml')}" />
+  <xacro:property
+    name="lidar_config"
+    value="${xacro.load_yaml('$(arg lidar_config_file)')['lidar']}" />
+  <!-- 기존 라이다 링크에 측정 기능 연결 -->
+  <gazebo reference="laser_frame">
+    <sensor name="lidar_sensor" type="gpu_lidar">
+      <pose>0 0 0 0 0 0</pose>
+      <always_on>true</always_on>
+      <update_rate>${lidar_config['update_rate_hz']}</update_rate>
+      <topic>/scan</topic>
+      <gz_frame_id>laser_frame</gz_frame_id>
+      <lidar>
+        <scan>
+          <horizontal>
+            <samples>${lidar_config['horizontal_samples']}</samples>
+            <resolution>1</resolution>
+            <min_angle>${lidar_config['min_angle_rad']}</min_angle>
+            <max_angle>${lidar_config['max_angle_rad']}</max_angle>
+          </horizontal>
+          <!-- 수평면 한 층을 측정하는 2D 라이다 -->
+          <vertical>
+            <samples>1</samples>
+            <resolution>1</resolution>
+            <min_angle>0</min_angle>
+            <max_angle>0</max_angle>
+          </vertical>
+        </scan>
+        <range>
+          <min>${lidar_config['min_range_m']}</min>
+          <max>${lidar_config['max_range_m']}</max>
+          <resolution>${lidar_config['range_resolution_m']}</resolution>
+        </range>
+      </lidar>
+    </sensor>
+  </gazebo>
 </robot>

Commit message: test(vehicle_description): validate odometry against Gazebo ground truth

File: src/vehicle_description/urdf/gazebo.xacro (robot description, xacro)
@@ -16,5 +16,5 @@
           이 설정은 바퀴 속도 명령과 오도메트리 계산에 모두 영향을 주므로,
           보정 후 직선·양방향 회전·사각형 주행을 재검증해야 한다. -->
-      <wheel_separation>${wheel_separation * 1.57}</wheel_separation>
+      <wheel_separation>${wheel_separation * wheel_separation_multiplier}</wheel_separation>
       <wheel_radius>${wheel_radius}</wheel_radius>
       <topic>/cmd_vel</topic>
@@ -23,4 +23,16 @@
       <child_frame_id>base_footprint</child_frame_id>
       <tf_topic>/tf</tf_topic>
+    </plugin>
+    <!-- 바퀴 회전량과 독립적으로 실제 모델 자세를 발행한다.
+         검증용 TF는 별도 토픽으로 분리하고 ROS /tf로 브리지하지 않는다. -->
+    <plugin filename="gz-sim-odometry-publisher-system"
+            name="gz::sim::systems::OdometryPublisher">
+      <odom_frame>world</odom_frame>
+      <robot_base_frame>base_footprint</robot_base_frame>
+      <odom_topic>/ground_truth/odom</odom_topic>
+      <tf_topic>/ground_truth/tf</tf_topic>
+      <dimensions>2</dimensions>
+      <odom_publish_frequency>50</odom_publish_frequency>
+      <gaussian_noise>0</gaussian_noise>
     </plugin>
   </gazebo>

File: src/vehicle_description/urdf/vehicle.urdf.xacro (robot description, xacro)
@@ -2,7 +2,16 @@
 <robot xmlns:xacro="http://www.ros.org/wiki/xacro" name="vehicle">
   <!-- 4wd_platform.stl에서 분리한 메시 기준, 단위 m. 원본 -Z가 전방, 네 바퀴 축의 중심이 원점. -->
+  <xacro:property
+    name="vehicle_config"
+    value="${xacro.load_yaml(
+      xacro.abs_filename('../config/vehicle.yaml'))['vehicle']}"/>
   <xacro:property name="wheel_radius" value="0.0335"/>
   <xacro:property name="wheel_width" value="0.027"/>
-  <xacro:property name="wheel_separation" value="0.1203"/>
+  <xacro:property
+    name="wheel_separation"
+    value="${vehicle_config['geometry']['wheel_separation_m']}"/>
+  <xacro:property
+    name="wheel_separation_multiplier"
+    value="${vehicle_config['calibration']['wheel_separation_multiplier']}"/>
   <xacro:property name="wheelbase" value="0.0994"/>
   <xacro:property name="chassis_center_x" value="-0.006"/>

Commit message: refactor(bringup): separate simulation and hardware backends

File: src/vehicle_description/urdf/gazebo.xacro (robot description, xacro)
@@ -3,4 +3,8 @@
   <xacro:arg name="safety_config_file"
     default="$(find vehicle_actuator_sim)/config/safety.yaml" />
+  <xacro:arg name="simulation_config_file"
+    default="$(find vehicle_simulation)/config/simulation.yaml"/>
+  <xacro:property name="wheel_separation_multiplier"
+    value="${xacro.load_yaml('$(arg simulation_config_file)')['simulation']['wheel_separation_multiplier']}"/>
   <gazebo>
     <plugin filename="gz-sim-joint-state-publisher-system"
@@ -42,5 +46,5 @@
   <xacro:arg
     name="lidar_config_file"
-    default="${xacro.abs_filename('../config/lidar.yaml')}" />
+    default="$(find vehicle_simulation)/config/lidar.yaml" />
   <xacro:property
     name="lidar_config"

File: src/vehicle_description/urdf/vehicle.urdf.xacro (robot description, xacro)
@@ -11,7 +11,5 @@
     name="wheel_separation"
     value="${vehicle_config['geometry']['wheel_separation_m']}"/>
-  <xacro:property
-    name="wheel_separation_multiplier"
-    value="${vehicle_config['calibration']['wheel_separation_multiplier']}"/>
+  <xacro:arg name="simulation" default="false"/>
   <xacro:property name="wheelbase" value="0.0994"/>
   <xacro:property name="chassis_center_x" value="-0.006"/>
@@ -25,5 +23,7 @@
   <xacro:include filename="sensors.xacro"/>
   <xacro:include filename="boards.xacro"/>
-  <xacro:include filename="gazebo.xacro"/>
+  <xacro:if value="$(arg simulation)">
+    <xacro:include filename="gazebo.xacro"/>
+  </xacro:if>
   <!-- 바닥 접지면에 놓이는 기준 좌표계 -->
   <link name="base_footprint"/>
